File: MiniDrive.kicad_pcb (KiCad board)
At the start: 2 copper layers, 25 x 40.1 mm, 22 parts, among them J1 Conn_LED, J2 Conn_24V, U1 TPS92200

Commit message: Change inductor to SMT
Parts:
- L1: footprint Inductor_THT:L_Radial_D8.7mm_P5.00mm_Fastron_07HCP -> Inductors:L_Wurth_WE-LQS-8040
- moved L1 2.57 mm to (147.0, 98.4)
Changed lines of the file:
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@@
+    )
+  )
+  (footprint "Inductors:L_Wurth_WE-LQS-8040" (layer "F.Cu")
+    (at 147 98.4 90)
+    (descr "Semi-Shielded High Saturation Power Inductor, body 4x4mm, https://www.we-online.com/catalog/en/WE-LQSH#/articles/WE-LQSH-4020")
+    (tags "SMT")
+    (property "Sheetfile" "MiniDrive.kicad_sch")
+    (property "Sheetname" "")
+    (property "ki_description" "Inductor")
+    (property "ki_keywords" "inductor choke coil reactor magnetic")
+    (attr smd)
+    (fp_text reference "L1" (at 5.15 0 unlocked) (layer "F.SilkS")
+        (effects (font (size 1 1) (thickness 0.15)))
+    )
+    (fp_text value "18 uH" (at 0 5.3 90 unlocked) (layer "F.Fab") hide
+        (effects (font (size 1 1) (thickness 0.15)))
+    )
+    (fp_text user "${REFERENCE}" (at 0 0 90 unlocked) (layer "F.Fab")
+        (effects (font (size 0.5 0.5) (thickness 0.075)))
+    )
+    (fp_line (start -4 4.1) (end 4 4.1)
+      (stroke (width 0.12) (type solid)) (layer "F.SilkS"))
+    (fp_line (start 0 -4.1) (end 4 -4.1)
+      (stroke (width 0.12) (type solid)) (layer "F.SilkS"))
+    (fp_rect (start -4.5 -4.3) (end 4.5 4.3)
+      (stroke (width 0.05) (type solid)) (fill none) (layer "F.CrtYd"))
+    (fp_line (start -4 -3) (end -4 4)
+      (stroke (width 0.1) (type solid)) (layer "F.Fab"))
+    (fp_line (start -4 4) (end 4 4)
+      (stroke (width 0.1) (type solid)) (layer "F.Fab"))
+    (fp_line (start -3 -4) (end -4 -3)
+      (stroke (width 0.1) (type solid)) (layer "F.Fab"))
+    (fp_line (start -3 -4) (end 4 -4)
+      (stroke (width 0.1) (type solid)) (layer "F.Fab"))
+    (fp_line (start 4 -4) (end 4 4)
+      (stroke (width 0.1) (type solid)) (layer "F.Fab"))
+    (pad "1" smd rect (at -3.1 0 90) (size 2.4 7.5) (layers "F.Cu" "F.Paste" "F.Mask")
+      (net 1 "Net-(U1-SW)") (pinfunction "1") (pintype "passive"))
+    (pad "2" smd rect (at 3.1 0 90) (size 2.4 7.5) (layers "F.Cu" "F.Paste" "F.Mask")
+      (net 9 "Net-(C4-Pad1)") (pinfunction "2") (pintype "passive"))
+    (model "${KICAD6_3DMODEL_DIR}/Inductor_SMD_Wurth.3dshapes/L_Wurth_WE-LQSH-4020.wrl"
+      (offset (xyz 0 0 0))
+      (scale (xyz 1 1 1))
+      (rotate (xyz 0 0 0))
     )
   )
@@
       (net 4 "GND") (pinfunction "1") (pintype "passive"))
   )
-  (footprint "Inductor_THT:L_Radial_D8.7mm_P5.00mm_Fastron_07HCP" (layer "F.Cu")
-    (at 147.5 100.925 90)
-    (descr "Inductor, Radial series, Radial, pin pitch=5.00mm, , diameter=8.7mm, Fastron, 07HCP, http://cdn-reichelt.de/documents/datenblatt/B400/DS_07HCP.pdf")
-    (tags "Inductor Radial series Radial pin pitch 5.00mm  diameter 8.7mm Fastron 07HCP")
-    (property "Sheetfile" "MiniDrive.kicad_sch")
-    (property "Sheetname" "")
-    (property "ki_description" "Inductor")
-    (property "ki_keywords" "inductor choke coil reactor magnetic")
-    (attr through_hole)
-    (fp_text reference "L1" (at -1.75 -3.5 180) (layer "F.SilkS")
-        (effects (font (size 1 1) (thickness 0.15)))
-    )
-    (fp_text value "18 uH" (at 2.5 5.6 90) (layer "F.Fab") hide
-        (effects (font (size 1 1) (thickness 0.15)))
-    )
-    (fp_text user "${REFERENCE}" (at 2.5 0 90) (layer "F.Fab")
-        (effects (font (size 1 1) (thickness 0.15)))
-    )
-    (fp_circle (center 2.5 0) (end 6.97 0)
-      (stroke (width 0.12) (type solid)) (fill none) (layer "F.SilkS"))
-    (fp_circle (center 2.5 0) (end 7.1 0)
-      (stroke (width 0.05) (type solid)) (fill none) (layer "F.CrtYd"))
-    (fp_circle (center 2.5 0) (end 6.85 0)
-      (stroke (width 0.1) (type solid)) (fill none) (layer "F.Fab"))
-    (pad "1" thru_hole circle (at 0 0 90) (size 2.6 2.6) (drill 1.3) (layers "*.Cu" "*.Mask")
-      (net 1 "Net-(U1-SW)") (pinfunction "1") (pintype "passive"))
-    (pad "2" thru_hole circle (at 5 0 90) (size 2.6 2.6) (drill 1.3) (layers "*.Cu" "*.Mask")
-      (net 9 "Net-(C4-Pad1)") (pinfunction "2") (pintype "passive"))
-    (model "${KICAD6_3DMODEL_DIR}/Inductor_THT.3dshapes/L_Radial_D8.7mm_P5.00mm_Fastron_07HCP.wrl"
-      (offset (xyz 0 0 0))
-      (scale (xyz 1 1 1))
-      (rotate (xyz 0 0 0))
-    )
-  )
   (footprint "MountingHole:MountingHole_2.7mm_M2.5" (layer "F.Cu")
     (at 131 86)
@@
   )
   (segment (start 138.35 100.95) (end 140.6725 100.95) (width 0.5) (layer "F.Cu") (net 1))
-  (segment (start 144.145 100.6225) (end 144.4475 100.925) (width 0.5) (layer "F.Cu") (net 1))
   (segment (start 140.6725 100.95) (end 141 100.6225) (width 0.5) (layer "F.Cu") (net 1))
   (segment (start 141 100.5625) (end 140.6125 100.95) (width 0.5) (layer "F.Cu") (net 1))
-  (segment (start 141 100.6225) (end 144.145 100.6225) (width 0.5) (layer "F.Cu") (net 1))
-  (segment (start 144.4475 100.925) (end 147.5 100.925) (width 0.5) (layer "F.Cu") (net 1))
+  (segment (start 147 101.5) (end 143.5 101.5) (width 0.5) (layer "F.Cu") (net 1))
+  (segment (start 143.5 101.5) (end 142.6225 100.6225) (width 0.5) (layer "F.Cu") (net 1))
+  (segment (start 142.6225 100.6225) (end 141 100.6225) (width 0.5) (layer "F.Cu") (net 1))
   (segment (start 138.35 100) (end 138.35 98.505) (width 0.5) (layer "F.Cu") (net 2))
   (segment (start 139.3575 97.4975) (end 141 97.4975) (width 0.5) (layer "F.Cu") (net 2))
@@
         (xy 137.16 114.935)
         (xy 129 114.935)
-        (xy 129 97.855)
-        (xy 134.27 97.855)
+        (xy 129 97.105)
+        (xy 134.27 97.105)
         (xy 134.27 101.085)
       )
@@
     (polygon
       (pts
-        (xy 140 96.5)
-        (xy 143.5 96.5)
-        (xy 143.5 98)
+        (xy 140 98)
         (xy 152.135 98)
-        (xy 152.135 86.19)
-        (xy 148.32 86.19)
-        (xy 148.32 93.175)
+        (xy 152.135 86)
+        (xy 148.07 86)
+        (xy 148.07 93.175)
         (xy 140 93.175)
       )

Commit message: Add power LED
Parts:
- added D1: LED, LED_SMD:LED_0603_1608Metric, F.Cu at (130.5, 115.2)
- added R6: 2k, Resistor_SMD:R_0805_2012Metric, F.Cu at (130.5, 118.5)
Routing:
- net +24V: track 9.96 -> 25.1 mm
- net Net-(D1-A): track 0.00 -> 1.55 mm
Other:
- board text added: "+"
- board text added: "-"
Changed lines of the file:
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@@
   (net 8 "Net-(U1-DIM)")
   (net 9 "Net-(C4-Pad1)")
+  (net 10 "Net-(D1-A)")
   (footprint "Package_TO_SOT_SMD:SOT-23-6_Handsoldering" (layer "F.Cu")
     (at 137 100.95)
@@
     )
   )
+  (footprint "Resistor_SMD:R_0805_2012Metric" (layer "F.Cu")
+    (at 130.5 118.5 90)
+    (descr "Resistor SMD 0805 (2012 Metric), square (rectangular) end terminal, IPC_7351 nominal, (Body size source: IPC-SM-782 page 72, https://www.pcb-3d.com/wordpress/wp-content/uploads/ipc-sm-782a_amendment_1_and_2.pdf), generated with kicad-footprint-generator")
+    (tags "resistor")
+    (property "Sheetfile" "MiniDrive.kicad_sch")
+    (property "Sheetname" "")
+    (property "ki_description" "Resistor")
+    (property "ki_keywords" "R res resistor")
+    (attr smd)
+    (fp_text reference "R6" (at -2.25 0 180) (layer "F.SilkS")
+        (effects (font (size 1 1) (thickness 0.15)))
+    )
+    (fp_text value "2k" (at 0 1.65 90) (layer "F.Fab") hide
+        (effects (font (size 1 1) (thickness 0.15)))
+    )
+    (fp_text user "${REFERENCE}" (at 0 0 90) (layer "F.Fab")
+        (effects (font (size 0.5 0.5) (thickness 0.08)))
+    )
+    (fp_line (start -0.227064 -0.735) (end 0.227064 -0.735)
+      (stroke (width 0.12) (type solid)) (layer "F.SilkS"))
+    (fp_line (start -0.227064 0.735) (end 0.227064 0.735)
+      (stroke (width 0.12) (type solid)) (layer "F.SilkS"))
+    (fp_line (start -1.68 -0.95) (end 1.68 -0.95)
+      (stroke (width 0.05) (type solid)) (layer "F.CrtYd"))
+    (fp_line (start -1.68 0.95) (end -1.68 -0.95)
+      (stroke (width 0.05) (type solid)) (layer "F.CrtYd"))
+    (fp_line (start 1.68 -0.95) (end 1.68 0.95)
+      (stroke (width 0.05) (type solid)) (layer "F.CrtYd"))
+    (fp_line (start 1.68 0.95) (end -1.68 0.95)
+      (stroke (width 0.05) (type solid)) (layer "F.CrtYd"))
+    (fp_line (start -1 -0.625) (end 1 -0.625)
+      (stroke (width 0.1) (type solid)) (layer "F.Fab"))
+    (fp_line (start -1 0.625) (end -1 -0.625)
+      (stroke (width 0.1) (type solid)) (layer "F.Fab"))
+    (fp_line (start 1 -0.625) (end 1 0.625)
+      (stroke (width 0.1) (type solid)) (layer "F.Fab"))
+    (fp_line (start 1 0.625) (end -1 0.625)
+      (stroke (width 0.1) (type solid)) (layer "F.Fab"))
+    (pad "1" smd roundrect (at -0.9125 0 90) (size 1.025 1.4) (layers "F.Cu" "F.Paste" "F.Mask") (roundrect_rratio 0.243902)
+      (net 3 "+24V") (pintype "passive"))
+    (pad "2" smd roundrect (at 0.9125 0 90) (size 1.025 1.4) (layers "F.Cu" "F.Paste" "F.Mask") (roundrect_rratio 0.243902)
+      (net 10 "Net-(D1-A)") (pintype "passive"))
+    (model "${KICAD6_3DMODEL_DIR}/Resistor_SMD.3dshapes/R_0805_2012Metric.wrl"
+      (offset (xyz 0 0 0))
+      (scale (xyz 1 1 1))
+      (rotate (xyz 0 0 0))
+    )
+  )
   (footprint "Capacitor_SMD:C_1206_3216Metric_Pad1.33x1.80mm_HandSolder" (layer "F.Cu")
     (at 137 107.5 180)
@@
     (pad "" np_thru_hole circle (at 0 0) (size 2.7 2.7) (drill 2.7) (layers "*.Cu" "*.Mask"))
   )
+  (footprint "LED_SMD:LED_0603_1608Metric" (layer "F.Cu")
+    (at 130.5 115.25 -90)
+    (descr "LED SMD 0603 (1608 Metric), square (rectangular) end terminal, IPC_7351 nominal, (Body size source: http://www.tortai-tech.com/upload/download/2011102023233369053.pdf), generated with kicad-footprint-generator")
+    (tags "LED")
+    (property "Sheetfile" "MiniDrive.kicad_sch")
+    (property "Sheetname" "")
+    (property "ki_description" "Light emitting diode")
+    (property "ki_keywords" "LED diode")
+    (attr smd)
+    (fp_text reference "D1" (at -2.2125 0 -180) (layer "F.SilkS")
+        (effects (font (size 1 1) (thickness 0.15)))
+    )
+    (fp_text value "LED" (at 0 1.43 90) (layer "F.Fab") hide
+        (effects (font (size 1 1) (thickness 0.15)))
+    )
+    (fp_text user "${REFERENCE}" (at 0 0 90) (layer "F.Fab")
+        (effects (font (size 0.4 0.4) (thickness 0.06)))
+    )
+    (fp_line (start -1.485 -0.735) (end -1.485 0.735)
+      (stroke (width 0.12) (type solid)) (layer "F.SilkS"))
+    (fp_line (start -1.485 0.735) (end 0.8 0.735)
+      (stroke (width 0.12) (type solid)) (layer "F.SilkS"))
+    (fp_line (start 0.8 -0.735) (end -1.485 -0.735)
+      (stroke (width 0.12) (type solid)) (layer "F.SilkS"))
+    (fp_line (start -1.48 -0.73) (end 1.48 -0.73)
+      (stroke (width 0.05) (type solid)) (layer "F.CrtYd"))
+    (fp_line (start -1.48 0.73) (end -1.48 -0.73)
+      (stroke (width 0.05) (type solid)) (layer "F.CrtYd"))
+    (fp_line (start 1.48 -0.73) (end 1.48 0.73)
+      (stroke (width 0.05) (type solid)) (layer "F.CrtYd"))
+    (fp_line (start 1.48 0.73) (end -1.48 0.73)
+      (stroke (width 0.05) (type solid)) (layer "F.CrtYd"))
+    (fp_line (start -0.8 -0.1) (end -0.8 0.4)
+      (stroke (width 0.1) (type solid)) (layer "F.Fab"))
+    (fp_line (start -0.8 0.4) (end 0.8 0.4)
+      (stroke (width 0.1) (type solid)) (layer "F.Fab"))
+    (fp_line (start -0.5 -0.4) (end -0.8 -0.1)
+      (stroke (width 0.1) (type solid)) (layer "F.Fab"))
+    (fp_line (start 0.8 -0.4) (end -0.5 -0.4)
+      (stroke (width 0.1) (type solid)) (layer "F.Fab"))
+    (fp_line (start 0.8 0.4) (end 0.8 -0.4)
+      (stroke (width 0.1) (type solid)) (layer "F.Fab"))
+    (pad "1" smd roundrect (at -0.7875 0 270) (size 0.875 0.95) (layers "F.Cu" "F.Paste" "F.Mask") (roundrect_rratio 0.25)
+      (net 4 "GND") (pinfunction "K") (pintype "passive"))
+    (pad "2" smd roundrect (at 0.7875 0 270) (size 0.875 0.95) (layers "F.Cu" "F.Paste" "F.Mask") (roundrect_rratio 0.25)
+      (net 10 "Net-(D1-A)") (pinfunction "A") (pintype "passive"))
+    (model "${KICAD6_3DMODEL_DIR}/LED_SMD.3dshapes/LED_0603_1608Metric.wrl"
+      (offset (xyz 0 0 0))
+      (scale (xyz 1 1 1))
+      (rotate (xyz 0 0 0))
+    )
+  )
   (footprint "Resistor_SMD:R_1206_3216Metric_Pad1.30x1.75mm_HandSolder" (layer "F.Cu")
     (at 144.272 108.585 -90)
@@
   (gr_rect (start 127.5 81.865) (end 152.5 122)
     (stroke (width 0.1) (type default)) (fill none) (layer "Edge.Cuts"))
-  (gr_text "MiniDrive LED Driver\nRevision 0" (at 130.81 121.92 90) (layer "F.SilkS")
-    (effects (font (size 1 1) (thickness 0.2) bold) (justify left bottom))
+  (gr_text "MiniDrive LED Driver\nRevision 0" (at 131 121.5 90) (layer "B.SilkS")
+    (effects (font (size 1 1) (thickness 0.2) bold) (justify right bottom mirror))
+  )
+  (gr_text "+" (at 138.75 111.25) (layer "F.SilkS")
+    (effects (font (size 1.5 1.5) (thickness 0.3) bold) (justify bottom))
+  )
+  (gr_text "-" (at 138.25 94) (layer "F.SilkS")
+    (effects (font (size 1.5 1.5) (thickness 0.3) bold) (justify bottom))
+  )
+  (gr_text "+" (at 141.75 94) (layer "F.SilkS")
+    (effects (font (size 1.5 1.5) (thickness 0.3) bold) (justify bottom))
   )
   (gr_text "LED Out" (at 128.905 83.185) (layer "F.SilkS")
@@
   (gr_text "Power In" (at 142.24 121.92) (layer "F.SilkS")
     (effects (font (size 1 1) (thickness 0.2) bold) (justify left bottom))
+  )
+  (gr_text "-" (at 135.25 111.25) (layer "F.SilkS")
+    (effects (font (size 1.5 1.5) (thickness 0.3) bold) (justify bottom))
   )
   (segment (start 138.35 100.95) (end 140.6725 100.95) (width 0.5) (layer "F.Cu") (net 1))
@@
   (segment (start 138.35 98.505) (end 139.3575 97.4975) (width 0.5) (layer "F.Cu") (net 2))
   (segment (start 138.6125 107.55) (end 138.5625 107.5) (width 0.25) (layer "F.Cu") (net 3))
+  (segment (start 139.5 115.5) (end 138.5 114.5) (width 0.25) (layer "F.Cu") (net 3))
+  (segment (start 139.5 117.75) (end 139.5 115.5) (width 0.25) (layer "F.Cu") (net 3))
+  (segment (start 137.8375 119.4125) (end 139.5 117.75) (width 0.25) (layer "F.Cu") (net 3))
   (segment (start 140.885 104.775) (end 140.61 104.5) (width 0.25) (layer "F.Cu") (net 3))
   (segment (start 140.61 104.5) (end 138.5625 104.5) (width 0.25) (layer "F.Cu") (net 3))
+  (segment (start 138.5 114.5) (end 138.5 112.68) (width 0.25) (layer "F.Cu") (net 3))
+  (segment (start 130.5 119.4125) (end 137.8375 119.4125) (width 0.25) (layer "F.Cu") (net 3))
   (segment (start 148.336 104.775) (end 140.885 104.775) (width 0.25) (layer "F.Cu") (net 3))
   (segment (start 137.12 96.3175) (end 137.12 101.38) (width 0.5) (layer "F.Cu") (net 4))
@@
   (segment (start 133.35 109.22) (end 134.265 110.135) (width 0.25) (layer "B.Cu") (net 8))
   (segment (start 134.265 110.135) (end 140.055 110.135) (width 0.25) (layer "B.Cu") (net 8))
+  (segment (start 130.5 117.5875) (end 130.5 116.0375) (width 0.25) (layer "F.Cu") (net 10))
   (zone (net 5) (net_name "Net-(J1-Pin_1)") (layer "F.Cu") (hatch edge 0.5)
     (priority 2)

Commit message: Add off-board dimming connector
Parts:
- removed TP3: V_DIM, TestPoint:TestPoint_THTPad_D1.5mm_Drill0.7mm
- added J3: Dimmer, Connector_JST:JST_PH_B2B-PH-K_1x02_P2.00mm_Vertical, F.Cu at (150.1, 110.2)
- moved TP1 1.91 mm to (146.5, 104.2)
- moved TP2 1.06 mm to (148.3, 106.2)
Routing:
- net GND: track 27.8 -> 36.0 mm
- net Net-(J3-Pin_2): track 28.2 -> 30.7 mm
- net +24V: track 25.1 -> 23.3 mm

Commit message: Change mounting holes to M3
Parts:
- H1, H2: footprint MountingHole:MountingHole_2.7mm_M2.5 -> MountingHole:MountingHole_3.2mm_M3
- moved H2 0.57 mm to (149.0, 118.5)
- moved H1 0.50 mm to (131.0, 85.5)
Changed lines of the file:
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@@
       (solder_mask_margin 0.25) (clearance 0.25))
   )
-  (footprint "MountingHole:MountingHole_2.7mm_M2.5" (layer "F.Cu")
-    (at 148.59 118.11)
-    (descr "Mounting Hole 2.7mm, no annular, M2.5")
-    (tags "mounting hole 2.7mm no annular m2.5")
+  (footprint "MountingHole:MountingHole_3.2mm_M3" (layer "F.Cu")
+    (at 149 118.5)
+    (descr "Mounting Hole 3.2mm, no annular, M3")
+    (tags "mounting hole 3.2mm no annular m3")
     (property "Sheetfile" "MiniDrive.kicad_sch")
     (property "Sheetname" "")
@@
     (property "ki_keywords" "mounting hole")
     (attr exclude_from_pos_files)
-    (fp_text reference "H2" (at 0 -2.286) (layer "F.SilkS") hide
-        (effects (font (size 1 1) (thickness 0.15)))
-    )
-    (fp_text value "MountingHole" (at 0 3.7) (layer "F.Fab") hide
+    (fp_text reference "H2" (at -4.5 0) (layer "F.SilkS") hide
+        (effects (font (size 1 1) (thickness 0.15)))
+    )
+    (fp_text value "MountingHole" (at 0 4.2) (layer "F.Fab") hide
         (effects (font (size 1 1) (thickness 0.15)))
     )
@@
         (effects (font (size 1 1) (thickness 0.15)))
     )
-    (fp_circle (center 0 0) (end 2.7 0)
+    (fp_circle (center 0 0) (end 3.2 0)
       (stroke (width 0.15) (type solid)) (fill none) (layer "Cmts.User"))
-    (fp_circle (center 0 0) (end 2.95 0)
-      (stroke (width 0.05) (type solid)) (fill none) (layer "F.CrtYd"))
-    (pad "" np_thru_hole circle (at 0 0) (size 2.7 2.7) (drill 2.7) (layers "*.Cu" "*.Mask"))
+    (fp_circle (center 0 0) (end 3.45 0)
+      (stroke (width 0.05) (type solid)) (fill none) (layer "F.CrtYd"))
+    (pad "" np_thru_hole circle (at 0 0) (size 3.2 3.2) (drill 3.2) (layers "F&B.Cu" "*.Mask"))
   )
   (footprint "LED_SMD:LED_0603_1608Metric" (layer "F.Cu")
@@
       (net 4 "GND") (pinfunction "1") (pintype "passive"))
   )
-  (footprint "MountingHole:MountingHole_2.7mm_M2.5" (layer "F.Cu")
-    (at 131 86)
-    (descr "Mounting Hole 2.7mm, no annular, M2.5")
-    (tags "mounting hole 2.7mm no annular m2.5")
+  (footprint "MountingHole:MountingHole_3.2mm_M3" (layer "F.Cu")
+    (at 131 85.5)
+    (descr "Mounting Hole 3.2mm, no annular, M3")
+    (tags "mounting hole 3.2mm no annular m3")
     (property "Sheetfile" "MiniDrive.kicad_sch")
     (property "Sheetname" "")
@@
     (property "ki_keywords" "mounting hole")
     (attr exclude_from_pos_files)
-    (fp_text reference "H1" (at 0 2.392) (layer "F.SilkS") hide
-        (effects (font (size 1 1) (thickness 0.15)))
-    )
-    (fp_text value "MountingHole" (at 0 3.7) (layer "F.Fab") hide
+    (fp_text reference "H1" (at 0 4) (layer "F.SilkS") hide
+        (effects (font (size 1 1) (thickness 0.15)))
+    )
+    (fp_text value "MountingHole" (at 0 4.2) (layer "F.Fab") hide
         (effects (font (size 1 1) (thickness 0.15)))
     )
@@
         (effects (font (size 1 1) (thickness 0.15)))
     )
-    (fp_circle (center 0 0) (end 2.7 0)
+    (fp_circle (center 0 0) (end 3.2 0)
       (stroke (width 0.15) (type solid)) (fill none) (layer "Cmts.User"))
-    (fp_circle (center 0 0) (end 2.95 0)
-      (stroke (width 0.05) (type solid)) (fill none) (layer "F.CrtYd"))
-    (pad "" np_thru_hole circle (at 0 0) (size 2.7 2.7) (drill 2.7) (layers "*.Cu" "*.Mask"))
+    (fp_circle (center 0 0) (end 3.45 0)
+      (stroke (width 0.05) (type solid)) (fill none) (layer "F.CrtYd"))
+    (pad "" np_thru_hole circle (at 0 0) (size 3.2 3.2) (drill 3.2) (layers "*.Cu" "*.Mask"))
   )
   (gr_rect (start 127.5 81.865) (end 152.5 122)
@@
     (effects (font (size 1 1) (thickness 0.2) bold) (justify right bottom mirror))
   )
-  (gr_text "+" (at 138.75 111.25) (layer "F.SilkS")
+  (gr_text "+" (at 140.5 113.5) (layer "F.SilkS")
     (effects (font (size 1.5 1.5) (thickness 0.3) bold) (justify bottom))
   )
-  (gr_text "-" (at 138.25 94) (layer "F.SilkS")
-    (effects (font (size 1.5 1.5) (thickness 0.3) bold) (justify bottom))
-  )
-  (gr_text "+" (at 141.75 94) (layer "F.SilkS")
-    (effects (font (size 1.5 1.5) (thickness 0.3) bold) (justify bottom))
+  (gr_text "-" (at 136.5 91) (layer "F.SilkS")
+    (effects (font (size 1.5 1.5) (thickness 0.3) bold))
+  )
+  (gr_text "+" (at 143.5 91) (layer "F.SilkS")
+    (effects (font (size 1.5 1.5) (thickness 0.3) bold))
   )
   (gr_text "LED Out" (at 128.905 83.185) (layer "F.SilkS")
@@
     (effects (font (size 1 1) (thickness 0.2) bold) (justify left bottom))
   )
-  (gr_text "-" (at 135.25 111.25) (layer "F.SilkS")
+  (gr_text "-" (at 133.5 113.5) (layer "F.SilkS")
     (effects (font (size 1.5 1.5) (thickness 0.3) bold) (justify bottom))
   )
