File: MiniDrive.kicad_sch (KiCad schematic)
At the start: 24 parts, among them J1 Conn_LED, J2 Conn_24V, J3 Dimmer, U1 TPS92200

Commit message: Clean up schematic and layout
Parts:
- removed TP4: TestPoint, TestPoint:TestPoint_THTPad_D1.5mm_Drill0.7mm, symbol Connector:TestPoint
- added F1: Polyfuse, Fuse:Fuse_1206_3216Metric, symbol Device:Polyfuse
- C1, C3: footprint Capacitor_SMD:C_1210_3225Metric_Pad1.33x2.70mm_HandSolder -> Capacitor_SMD:C_1210_3225Metric
- C2, C4: footprint Capacitor_SMD:C_1206_3216Metric_Pad1.33x1.80mm_HandSolder -> Capacitor_SMD:C_1206_3216Metric
- C5: footprint Capacitor_SMD:C_0402_1005Metric_Pad0.74x0.62mm_HandSolder -> Capacitor_SMD:C_0402_1005Metric
- R1, R2, R3, R4, R5: footprint Resistor_SMD:R_1206_3216Metric_Pad1.30x1.75mm_HandSolder -> Resistor_SMD:R_0805_2012Metric
- U1: footprint Package_TO_SOT_SMD:SOT-23-6_Handsoldering -> Package_TO_SOT_SMD:SOT-23-6
- renumbered TP5 to TP3
Connections:
- net at R1.2, R2.1: now also F1.1; no longer J1.1 (Pin_1)
- new net: F1.2, J1.1 (Pin_1)
Other:
- note added: "Vf for D1 is 3.2V, so R6 sees 20.8V. Total power dissipated by R6 is only 206-228 mW."
- moved on the sheet: C1, C2, C3, C4, C5, D1, H1, H2, J1, J2, J3, L1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

Commit message: Revert back to 1206 resistors
Parts:
- R1, R2, R3, R4, R5: footprint Resistor_SMD:R_0805_2012Metric -> Resistor_SMD:R_1206_3216Metric
Changed lines of the file:
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@@
       (effects (font (size 1.27 1.27)) (justify right))
     )
-    (property "Footprint" "Resistor_SMD:R_0805_2012Metric" (at 77.343 76.835 90)
+    (property "Footprint" "Resistor_SMD:R_1206_3216Metric" (at 77.343 76.835 90)
       (effects (font (size 1.27 1.27)) hide)
     )
@@
       (effects (font (size 1.27 1.27)) (justify right))
     )
-    (property "Footprint" "Resistor_SMD:R_0805_2012Metric" (at 77.343 106.045 90)
+    (property "Footprint" "Resistor_SMD:R_1206_3216Metric" (at 77.343 106.045 90)
       (effects (font (size 1.27 1.27)) hide)
     )
@@
       (effects (font (size 1.27 1.27)) (justify right))
     )
-    (property "Footprint" "Resistor_SMD:R_0805_2012Metric" (at 223.393 97.155 90)
+    (property "Footprint" "Resistor_SMD:R_1206_3216Metric" (at 223.393 97.155 90)
       (effects (font (size 1.27 1.27)) hide)
     )
@@
       (effects (font (size 1.27 1.27)))
     )
-    (property "Footprint" "Resistor_SMD:R_0805_2012Metric" (at 191.77 85.217 90)
+    (property "Footprint" "Resistor_SMD:R_1206_3216Metric" (at 191.77 85.217 90)
       (effects (font (size 1.27 1.27)) hide)
     )
@@
       (effects (font (size 1.27 1.27)))
     )
-    (property "Footprint" "Resistor_SMD:R_0805_2012Metric" (at 225.425 53.467 90)
-      (effects (font (size 1.27 1.27)) hide)
-    )
+    (property "Footprint" "Resistor_SMD:R_1206_3216Metric" (at 225.425 53.467 90)
+      (effects (font (size 1.27 1.27)) hide)
+    )

Commit message: Minor tweaks, remove F1
Parts:
- removed F1: Polyfuse, Fuse:Fuse_1206_3216Metric, symbol Device:Polyfuse
- J3: now not fitted
Connections:
- net at J1.1 (Pin_1): now also R1.2, R2.1
Changed lines of the file:
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@@
-    (stroke (width 0) (type default))
-  )
-  (wire (pts (xy 221.615 73.66) (xy 221.615 86.995))
     (stroke (width 0) (type default))
   )
@@
     (stroke (width 0) (type default))
   )
-  (wire (pts (xy 221.615 57.785) (xy 221.615 66.04))
+  (wire (pts (xy 221.615 57.785) (xy 221.615 86.995))
     (stroke (width 0) (type default))
   )
@@
   )
   (symbol (lib_id "Connector_Generic:Conn_01x02") (at 45.085 95.885 180) (unit 1)
-    (in_bom yes) (on_board yes) (dnp no) (fields_autoplaced)
+    (in_bom yes) (on_board yes) (dnp yes) (fields_autoplaced)
     (property "Reference" "J3" (at 45.085 86.995 0)
       (effects (font (size 1.27 1.27)))
@@
         )
       )
-    )
-  )
-  (symbol (lib_id "Device:Polyfuse") (at 221.615 69.85 180) (unit 1)
-    (in_bom yes) (on_board yes) (dnp no) (fields_autoplaced)
-    (property "Reference" "F1" (at 224.155 68.58 0)
-      (effects (font (size 1.27 1.27)) (justify right))
-    )
-    (property "Value" "Polyfuse" (at 224.155 71.12 0)
-      (effects (font (size 1.27 1.27)) (justify right))
-    )
-    (property "Footprint" "Fuse:Fuse_1206_3216Metric" (at 220.345 64.77 0)
-      (effects (font (size 1.27 1.27)) (justify left) hide)
-    )
-    (property "Datasheet" "~" (at 221.615 69.85 0)
-      (effects (font (size 1.27 1.27)) hide)
-    )
-    (pin "1")
-    (pin "2")
-    (instances
-      (project "MiniDrive"
-        (path "/e06caad1-a246-4f16-9d4f-053507cbe732"
-          (reference "F1") (unit 1)
-        )
-      )
